File: KiCad/GR_DTMF_Decoder.kicad_pcb (KiCad board)
At the start: 2 copper layers, 67.1 x 26.3 mm, 17 parts, among them J1 Conn_01x02, J2 Conn_01x02, J3 Conn_01x07, J4 RJ12, T1 SM-LP-5001E, U1 MT88L70AS1, Y1 3.579545 MHz

Commit message: Add files via upload
Parts:
- added R4: 10K, Resistor_SMD:R_0805_2012Metric_Pad1.15x1.40mm_HandSolder, F.Cu at (146.3, 106.6)
- added R5: 10K, Resistor_SMD:R_0805_2012Metric_Pad1.15x1.40mm_HandSolder, F.Cu at (138.2, 108.6)
- Z1, Z2: value 3V3 -> 2V4
- moved R1 4.40 mm to (142.3, 106.6), turned to 180 degrees
- moved C2 1.47 mm to (138.3, 110.7), turned to 180 degrees
Connections:
- R1 pad 2: Net-(C2-Pad1) -> Net-(R1-Pad2)
Routing:
- net Net-(R1-Pad2): track 0.00 -> 18.4 mm, vias 0 -> 2
- net Net-(R4-Pad2): track 9.03 -> 14.1 mm
- net Net-(C2-Pad2): track 31.2 -> 29.6 mm
Other:
- board text added: "K"
