File: KiCad/GR_DTMF_Decoder.sch (KiCad schematic (older format))
At the start: 16 parts, among them J1 Conn_01x02, J2 Conn_01x02, J3 Conn_01x07, J4 RJ12, T1 SM-LP-5001E, U1 MT88L70AS1, Y1 3.579545 MHz

Commit message: Add files via upload
Parts:
- added R4, R5: 10K, Resistor_SMD:R_0805_2012Metric_Pad1.15x1.40mm_HandSolder, symbol Device:R_Small_US
- Z1, Z2: value 3V3 -> 2V4
Connections:
- wire segments 70 -> 75
Other:
- moved on the sheet: C2
Changed lines of the file:
@@
 L Device:C_Small C2
 U 1 1 62CE88D4
-P 5000 3125
-F 0 "C2" V 4771 3125 50  0000 C CNN
-F 1 "100nF" V 4862 3125 50  0000 C CNN
-F 2 "Capacitor_SMD:C_0805_2012Metric_Pad1.15x1.40mm_HandSolder" H 5000 3125 50  0001 C CNN
-F 3 "~" H 5000 3125 50  0001 C CNN
-	1    5000 3125
+P 4600 3125
+F 0 "C2" V 4371 3125 50  0000 C CNN
+F 1 "100nF" V 4462 3125 50  0000 C CNN
+F 2 "Capacitor_SMD:C_0805_2012Metric_Pad1.15x1.40mm_HandSolder" H 4600 3125 50  0001 C CNN
+F 3 "~" H 4600 3125 50  0001 C CNN
+	1    4600 3125
 	0    1    1    0
 $EndComp
@@
 U 1 1 62CEADE9
 P 5425 3125
-F 0 "R1" V 5220 3125 50  0000 C CNN
-F 1 "100K" V 5311 3125 50  0000 C CNN
+F 0 "R1" V 5500 3100 50  0000 C CNN
+F 1 "100K" V 5575 3150 50  0000 C CNN
 F 2 "Resistor_SMD:R_0805_2012Metric_Pad1.15x1.40mm_HandSolder" H 5425 3125 50  0001 C CNN
 F 3 "~" H 5425 3125 50  0001 C CNN
@@
 	5675 2425 5675 2250
 Wire Wire Line
-	5100 3125 5325 3125
+	4700 3125 4850 3125
 Wire Wire Line
 	5975 3325 6075 3325
@@
 P 4175 3375
 F 0 "Z1" V 4228 3272 60  0000 R CNN
-F 1 "3V3" V 4122 3272 60  0000 R CNN
+F 1 "2V4" V 4122 3272 60  0000 R CNN
 F 2 "footprints:Zener_MiniMELF" H 4375 3575 60  0001 L CNN
 F 3 "" H 4375 3675 60  0001 L CNN
@@
 Connection ~ 4175 3125
 Wire Wire Line
-	4175 3125 4900 3125
+	4175 3125 4500 3125
 Wire Wire Line
 	4175 3650 4175 3575
@@
 P 4175 3850
 F 0 "Z2" V 4100 4075 60  0000 R CNN
-F 1 "3V3" V 4200 4125 60  0000 R CNN
+F 1 "2V4" V 4200 4125 60  0000 R CNN
 F 2 "footprints:Zener_MiniMELF" H 4375 4050 60  0001 L CNN
 F 3 "" H 4375 4150 60  0001 L CNN
@@
 Wire Wire Line
 	5675 2725 5675 2675
+$Comp
+L Device:R_Small_US R5
+U 1 1 65F7BB0B
+P 4950 3125
+F 0 "R5" V 4850 3125 50  0000 C CNN
+F 1 "10K" V 5050 3125 50  0000 C CNN
+F 2 "Resistor_SMD:R_0805_2012Metric_Pad1.15x1.40mm_HandSolder" H 4950 3125 50  0001 C CNN
+F 3 "~" H 4950 3125 50  0001 C CNN
+	1    4950 3125
+	0    1    1    0
+$EndComp
+Wire Wire Line
+	5050 3125 5175 3125
+$Comp
+L Device:R_Small_US R4
+U 1 1 65F7C8B3
+P 5425 3025
+F 0 "R4" V 5575 3050 50  0000 C CNN
+F 1 "10K" V 5500 3025 50  0000 C CNN
+F 2 "Resistor_SMD:R_0805_2012Metric_Pad1.15x1.40mm_HandSolder" H 5425 3025 50  0001 C CNN
+F 3 "~" H 5425 3025 50  0001 C CNN
+	1    5425 3025
+	0    -1   -1   0
+$EndComp
+Wire Wire Line
+	5525 3025 5900 3025
+Connection ~ 5900 3025
+Wire Wire Line
+	5325 3025 5175 3025
+Wire Wire Line
+	5175 3025 5175 3125
+Connection ~ 5175 3125
+Wire Wire Line
+	5175 3125 5325 3125
 $EndSCHEMATC
